File: ADSCP/ADSCP.kicad_sch (KiCad schematic)
At the start: 0 parts

Commit message: edit schematic
Other:
- sheet Input Buffer and VI Converter（SSI2164 input） renamed Input Buffer and VI Converter
- added sheet Blend & Output (blend_and_output.kicad_sch)
- added sheet Sidechain 1 - Summing & Rectifier (sidechain1.kicad_sch)
- note added: "Audio path schematics"
- note added: "Side chain schematics"
Changed lines of the file:
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@@
 		(title "AI-Designed-Stereo-Compressor-Preamp")
+	)
+	(rectangle
+		(start 25.4 93.98)
+		(end 212.09 130.81)
+		(stroke
+			(width 1)
+			(type solid)
+		)
+		(fill
+			(type none)
+		)
+	)
+	(rectangle
+		(start 25.4 148.59)
+		(end 170.18 185.42)
+		(stroke
+			(width 1)
+			(type solid)
+		)
+		(fill
+			(type none)
+		)
 	)
 	(text "Let's build the ultimate Stereo Compressor / Preamp with the help of generative AI!!!"
@@
 		)
 	)
+	(text "Audio path schematics"
+		(exclude_from_sim no)
+		(at 61.214 88.9 0)
+		(effects
+			(font
+				(size 4 4)
+				(thickness 0.8)
+				(bold yes)
+			)
+		)
+	)
 	(text "https://github.com/ijnekenamay/AI-Designed-Stereo-Compressor-Preamp/"
 		(exclude_from_sim no)
@@
 				(bold yes)
 				(color 0 0 0 1)
+			)
+		)
+	)
+	(text "Side chain schematics"
+		(exclude_from_sim no)
+		(at 59.69 143.256 0)
+		(effects
+			(font
+				(size 4 4)
+				(thickness 0.8)
+				(bold yes)
 			)
 		)
@@
 	)
 	(sheet
-		(at 105.41 104.14)
+		(at 41.91 158.75)
+		(size 25.4 17.78)
+		(exclude_from_sim no)
+		(in_bom yes)
+		(on_board yes)
+		(dnp no)
+		(stroke
+			(width 0.1524)
+			(type solid)
+		)
+		(fill
+			(color 0 0 0 0.0000)
+		)
+		(property "Sheetname" "Sidechain 1 - Summing & Rectifier"
+			(at 29.972 156.972 0)
+			(effects
+				(font
+					(size 2 2)
+					(thickness 0.4)
+					(bold yes)
+				)
+				(justify left bottom)
+			)
+		)
+		(property "Sheetfile" "sidechain1.kicad_sch"
+			(at 41.148 177.8 0)
+			(effects
+				(font
+					(size 1.27 1.27)
+				)
+				(justify left top)
+			)
+		)
+		(instances
+			(project "ADSCP"
+				(path "/132f4570-4169-4ecf-b1f3-d724b5ad1d4e"
+					(page "6")
+				)
+			)
+		)
+	)
+	(sheet
+		(at 168.91 104.14)
+		(size 29.21 17.78)
+		(exclude_from_sim no)
+		(in_bom yes)
+		(on_board yes)
+		(dnp no)
+		(stroke
+			(width 0.1524)
+			(type solid)
+		)
+		(fill
+			(color 0 0 0 0.0000)
+		)
+		(property "Sheetname" "Blend & Output"
+			(at 171.196 102.108 0)
+			(effects
+				(font
+					(size 2 2)
+					(thickness 0.4)
+					(bold yes)
+				)
+				(justify left bottom)
+			)
+		)
+		(property "Sheetfile" "blend_and_output.kicad_sch"
+			(at 168.91 122.5046 0)
+			(effects
+				(font
+					(size 1.27 1.27)
+				)
+				(justify left top)
+			)
+		)
+		(instances
+			(project "ADSCP"
+				(path "/132f4570-4169-4ecf-b1f3-d724b5ad1d4e"
+					(page "5")
+				)
+			)
+		)
+	)
+	(sheet
+		(at 83.82 104.14)
 		(size 27.94 17.78)
 		(exclude_from_sim no)
@@
 		)
 		(property "Sheetname" "SSI2164 VCA Core"
-			(at 105.41 102.108 0)
+			(at 83.82 102.108 0)
 			(effects
 				(font
@@
 		)
 		(property "Sheetfile" "SSI2164.kicad_sch"
-			(at 105.41 122.5046 0)
+			(at 83.82 122.5046 0)
 			(effects
 				(font
@@
 			(color 0 0 0 0.0000)
 		)
-		(property "Sheetname" "Input Buffer and VI Converter（SSI2164 input）"
-			(at 24.384 102.362 0)
+		(property "Sheetname" "Input Buffer and VI Converter"
+			(at 32.766 101.854 0)
 			(effects
 				(font
@@
 	)
 	(sheet
-		(at 154.94 104.14)
+		(at 127 104.14)
 		(size 27.94 17.78)
 		(exclude_from_sim no)
@@
 		)
 		(property "Sheetname" "IV Converter & Make-up Gain"
-			(at 147.574 102.108 0)
+			(at 119.634 102.108 0)
 			(effects
 				(font
@@
 		)
 		(property "Sheetfile" "ivc_mug.kicad_sch"
-			(at 154.94 122.5046 0)
-			(effects
-				(font
+			(at 127 122.5046 0)
+			(effects
+				(font
