File: ADSCP/inputbuffer.kicad_sch (KiCad schematic)
At the start: 14 parts, among them J1 Input_Jack_L, J2 Input_Jack_R, U1 TL074 or OPA1644, U3 Opamp_Quad

Commit message: edit schematic
Parts:
- removed unit 3 of U1
- removed unit 4 of U1
- removed unit 3 of U3
- removed unit 4 of U3
- removed unit 2 of U3
- added U4: TL074, symbol Device:Opamp_Quad
- U3: value Opamp_Quad -> TL074 or OPA1644
Connections:
- net +15V: now also U4.4 (V+)
- net -15V: now also U4.11 (V-)
- net TO_BLEND_DRY_L renamed BLEND_DRY_L
- net TO_BLEND_DRY_R renamed BLEND_DRY_R
Other:
- moved on the sheet: U3E
