File: ADSCP/ivc_mug.kicad_sch (KiCad schematic)
At the start: 7 parts, among them U1 TL074 or OPA1644, U4 TL074 or OPA1644

Commit message: edit schematic
Parts:
- added C8: 47pF, Capacitor_THT:C_Disc_D4.3mm_W1.9mm_P5.00mm, symbol Device:C
- added MakeUpGain_R: 100kB, Connector_PinHeader_2.54mm:PinHeader_1x03_P2.54mm_Vertical, symbol Device:R_Potentiometer
- added R12, R14: 10k, Resistor_THT:R_Axial_DIN0207_L6.3mm_D2.5mm_P2.54mm_Vertical, symbol Device:R
- added R13: 20k, Resistor_THT:R_Axial_DIN0207_L6.3mm_D2.5mm_P2.54mm_Vertical, symbol Device:R
- added U3: TL074 or OPA1644, symbol Device:Opamp_Quad
- MakeUpGain_L: renamed from RV1; value R_Potentiometer -> 100kB; footprint (none) -> Connector_PinHeader_2.54mm:PinHeader_1x03_P2.54mm_Vertical
- renumbered U4 to U1
Connections:
- net GND: now also U3.10 (+), U3.5 (+)
- net IV_OUT_L: now also R10.2; no longer R10.1, R11.1
- net MAKEUP_OUT_L: now also R11.1; no longer MakeUpGain_L.3
- net at MakeUpGain_L.2, U1.9 (-): now also R10.1; no longer R11.2
- net at MakeUpGain_L.1: now also MakeUpGain_L.3, R11.2; no longer R10.2
- new net: MakeUpGain_R.1, MakeUpGain_R.3, R14.2
- new net: MakeUpGain_R.2, R12.1, U3.9 (-)
- new net IV_OUT_R: C8.1, R12.2, R13.2, U3.7
- new net MAKEUP_OUT_R: R14.1, U3.8
- new net VCA_OUT_R_TO_IV: C8.2, R13.1, U3.6 (-)
Other:
- moved on the sheet: MakeUpGain_L, R10, R11, U1C
